File: Supply.kicad_sch (KiCad schematic)
At the start: 27 parts

Commit message: PCB work 12/3
Parts:
- C15, C16, C17, C18, C19, C20: renamed from C?; footprint (none) -> Capacitor_SMD:C_0805_2012Metric_Pad1.18x1.45mm_HandSolder
- JP1: renamed from JP?; footprint (none) -> Connector_PinHeader_2.54mm:PinHeader_1x02_P2.54mm_Vertical
- L1: renamed from L?; footprint (none) -> Inductor_SMD:L_Coilcraft_LPS4018
- R15, R16, R17, R18, R19, R20, R21, R22, R23, R24, R25, R26, R27: renamed from R?; footprint (none) -> Resistor_SMD:R_0805_2012Metric_Pad1.20x1.40mm_HandSolder
- SW1, SW2: renamed from SW?; footprint (none) -> Button_Switch_THT:SW_DIP_SPSTx05_Slide_9.78x14.88mm_W7.62mm_P2.54mm
- U10, U9: renamed from U?; footprint (none) -> Package_DFN_QFN:DFN-8-1EP_3x3mm_P0.65mm_EP1.7x2.05mm
- U8: renamed from U?; footprint (none) -> JRIX TDFN Footprints:Package_TDFN-12_3x3mm_P0.4mm_IC_1.7x2.45mm
- gave numbers to parts that had none: 1
Connections:
- net GND: now also U10.4 (NC), U10.5 (NC), U10.9 (EPAD), U9.4 (NC), U9.5 (NC), U9.9 (EPAD); no longer U10.EPAD, U10.NC (5), U9.EPAD, U9.NC (5)
Other:
- moved on the sheet: C20, U10, U9
