File: VABCheck.kicad_sch (KiCad schematic)
At the start: 13 parts

Commit message: PCB work 12/3
Parts:
- C21: renamed from C?; footprint (none) -> Capacitor_SMD:C_0805_2012Metric_Pad1.18x1.45mm_HandSolder
- D6: renamed from D?; footprint (none) -> JRIX LED SMD:0603_1.6x0.8mm_dual_kingbright_APHB1608LG3R2C-AMT
- Q1: renamed from Q?; footprint (none) -> Package_TO_SOT_SMD:SOT-363_SC-70-6
- R28, R29, R30: renamed from R?; footprint (none) -> Resistor_SMD:R_0805_2012Metric_Pad1.20x1.40mm_HandSolder
- R31: renamed from R?; value 560R -> 1k6; footprint (none) -> Resistor_SMD:R_0805_2012Metric_Pad1.20x1.40mm_HandSolder
- R32: renamed from R?; value 560R -> 1k2; footprint (none) -> Resistor_SMD:R_0805_2012Metric_Pad1.20x1.40mm_HandSolder
- U11: renamed from U?; footprint (none) -> JRIX UDFN Footprints:Package_UDFN-6_1.2x1.0mm_P0.4
- gave numbers to parts that had none: 1
Changed lines of the file:
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@@
   (symbol (lib_id "Device:R_Small") (at 106.045 98.425 90) (unit 1)
     (in_bom yes) (on_board yes) (fields_autoplaced)
-    (property "Reference" "R?" (id 0) (at 106.045 92.71 90))
+    (property "Reference" "R30" (id 0) (at 106.045 92.71 90))
     (property "Value" "10k" (id 1) (at 106.045 95.25 90))
-    (property "Footprint" "" (id 2) (at 106.045 98.425 0)
+    (property "Footprint" "Resistor_SMD:R_0805_2012Metric_Pad1.20x1.40mm_HandSolder" (id 2) (at 106.045 98.425 0)
       (effects (font (size 1.27 1.27)) hide)
     )
@@
   (symbol (lib_id "power:GND") (at 33.02 103.505 0) (unit 1)
     (in_bom yes) (on_board yes) (fields_autoplaced)
-    (property "Reference" "#PWR?" (id 0) (at 33.02 109.855 0)
+    (property "Reference" "#PWR048" (id 0) (at 33.02 109.855 0)
       (effects (font (size 1.27 1.27)) hide)
     )
@@
   (symbol (lib_id "power:GND") (at 119.38 105.41 0) (unit 1)
     (in_bom yes) (on_board yes) (fields_autoplaced)
-    (property "Reference" "#PWR?" (id 0) (at 119.38 111.76 0)
+    (property "Reference" "#PWR051" (id 0) (at 119.38 111.76 0)
       (effects (font (size 1.27 1.27)) hide)
     )
@@
   (symbol (lib_id "JRIX LED:APHB1608LG3R2C") (at 111.76 65.405 90) (unit 1)
     (in_bom yes) (on_board yes) (fields_autoplaced)
-    (property "Reference" "D?" (id 0) (at 123.19 55.3719 90)
+    (property "Reference" "D6" (id 0) (at 123.19 55.3719 90)
       (effects (font (size 1.27 1.27)) (justify right))
     )
@@
       (effects (font (size 1.27 1.27)) (justify right))
     )
-    (property "Footprint" "" (id 2) (at 105.41 83.185 0)
+    (property "Footprint" "JRIX LED SMD:0603_1.6x0.8mm_dual_kingbright_APHB1608LG3R2C-AMT" (id 2) (at 105.41 83.185 0)
       (effects (font (size 1.27 1.27)) hide)
     )
@@
   (symbol (lib_id "power:GND") (at 114.3 86.995 0) (unit 1)
     (in_bom yes) (on_board yes) (fields_autoplaced)
-    (property "Reference" "#PWR?" (id 0) (at 114.3 93.345 0)
+    (property "Reference" "#PWR050" (id 0) (at 114.3 93.345 0)
       (effects (font (size 1.27 1.27)) hide)
     )
@@
   (symbol (lib_id "power:GND") (at 52.07 54.61 0) (unit 1)
     (in_bom yes) (on_board yes) (fields_autoplaced)
-    (property "Reference" "#PWR?" (id 0) (at 52.07 60.96 0)
+    (property "Reference" "#PWR049" (id 0) (at 52.07 60.96 0)
       (effects (font (size 1.27 1.27)) hide)
     )
@@
   (symbol (lib_id "JRIX Transistor:SIA931DJ") (at 81.28 71.12 270) (mirror x) (unit 1)
     (in_bom yes) (on_board yes) (fields_autoplaced)
-    (property "Reference" "Q?" (id 0) (at 81.28 57.15 90))
+    (property "Reference" "Q1" (id 0) (at 81.28 57.15 90))
     (property "Value" "SIA931DJ" (id 1) (at 81.28 59.69 90))
-    (property "Footprint" "" (id 2) (at 88.9 86.36 0)
+    (property "Footprint" "Package_TO_SOT_SMD:SOT-363_SC-70-6" (id 2) (at 88.9 86.36 0)
       (effects (font (size 1.27 1.27)) hide)
     )
@@
   (symbol (lib_id "Device:R_Small") (at 114.3 40.64 0) (unit 1)
     (in_bom yes) (on_board yes) (fields_autoplaced)
-    (property "Reference" "R?" (id 0) (at 116.84 39.3699 0)
-      (effects (font (size 1.27 1.27)) (justify left))
-    )
-    (property "Value" "560R" (id 1) (at 116.84 41.9099 0)
-      (effects (font (size 1.27 1.27)) (justify left))
-    )
-    (property "Footprint" "" (id 2) (at 114.3 40.64 0)
+    (property "Reference" "R31" (id 0) (at 116.84 39.3699 0)
+      (effects (font (size 1.27 1.27)) (justify left))
+    )
+    (property "Value" "1k6" (id 1) (at 116.84 41.9099 0)
+      (effects (font (size 1.27 1.27)) (justify left))
+    )
+    (property "Footprint" "Resistor_SMD:R_0805_2012Metric_Pad1.20x1.40mm_HandSolder" (id 2) (at 114.3 40.64 0)
       (effects (font (size 1.27 1.27)) hide)
     )
@@
   (symbol (lib_id "Device:R_Small") (at 68.58 90.17 0) (unit 1)
     (in_bom yes) (on_board yes) (fields_autoplaced)
-    (property "Reference" "R?" (id 0) (at 71.12 88.8999 0)
+    (property "Reference" "R29" (id 0) (at 71.12 88.8999 0)
       (effects (font (size 1.27 1.27)) (justify left))
     )
@@
       (effects (font (size 1.27 1.27)) (justify left))
     )
-    (property "Footprint" "" (id 2) (at 68.58 90.17 0)
+    (property "Footprint" "Resistor_SMD:R_0805_2012Metric_Pad1.20x1.40mm_HandSolder" (id 2) (at 68.58 90.17 0)
       (effects (font (size 1.27 1.27)) hide)
     )
@@
   (symbol (lib_id "Device:R_Small") (at 68.58 67.945 0) (unit 1)
     (in_bom yes) (on_board yes) (fields_autoplaced)
-    (property "Reference" "R?" (id 0) (at 71.12 66.6749 0)
+    (property "Reference" "R28" (id 0) (at 71.12 66.6749 0)
       (effects (font (size 1.27 1.27)) (justify left))
     )
@@
       (effects (font (size 1.27 1.27)) (justify left))
     )
-    (property "Footprint" "" (id 2) (at 68.58 67.945 0)
+    (property "Footprint" "Resistor_SMD:R_0805_2012Metric_Pad1.20x1.40mm_HandSolder" (id 2) (at 68.58 67.945 0)
       (effects (font (size 1.27 1.27)) hide)
     )
@@
   (symbol (lib_id "Transistor_BJT:BC846BPDW1") (at 116.84 98.425 0) (mirror x) (unit 2)
     (in_bom yes) (on_board yes) (fields_autoplaced)
-    (property "Reference" "Q?" (id 0) (at 121.92 97.1549 0)
+    (property "Reference" "Q2" (id 0) (at 121.92 97.1549 0)
       (effects (font (size 1.27 1.27)) (justify left))
     )
@@
   (symbol (lib_id "Device:C_Small") (at 43.18 43.815 0) (unit 1)
     (in_bom yes) (on_board yes) (fields_autoplaced)
-    (property "Reference" "C?" (id 0) (at 45.72 42.5512 0)
+    (property "Reference" "C21" (id 0) (at 45.72 42.5512 0)
       (effects (font (size 1.27 1.27)) (justify left))
     )
@@
       (effects (font (size 1.27 1.27)) (justify left))
     )
-    (property "Footprint" "" (id 2) (at 43.18 43.815 0)
+    (property "Footprint" "Capacitor_SMD:C_0805_2012Metric_Pad1.18x1.45mm_HandSolder" (id 2) (at 43.18 43.815 0)
       (effects (font (size 1.27 1.27)) hide)
     )
@@
   (symbol (lib_id "Device:R_Small") (at 119.38 40.64 0) (unit 1)
     (in_bom yes) (on_board yes) (fields_autoplaced)
-    (property "Reference" "R?" (id 0) (at 121.92 39.3699 0)
-      (effects (font (size 1.27 1.27)) (justify left))
-    )
-    (property "Value" "560R" (id 1) (at 121.92 41.9099 0)
-      (effects (font (size 1.27 1.27)) (justify left))
-    )
-    (property "Footprint" "" (id 2) (at 119.38 40.64 0)
+    (property "Reference" "R32" (id 0) (at 121.92 39.3699 0)
+      (effects (font (size 1.27 1.27)) (justify left))
+    )
+    (property "Value" "1k2" (id 1) (at 121.92 41.9099 0)
+      (effects (font (size 1.27 1.27)) (justify left))
+    )
+    (property "Footprint" "Resistor_SMD:R_0805_2012Metric_Pad1.20x1.40mm_HandSolder" (id 2) (at 119.38 40.64 0)
       (effects (font (size 1.27 1.27)) hide)
     )
@@
   (symbol (lib_id "Transistor_BJT:BC846BPDW1") (at 111.76 80.645 0) (unit 1)
     (in_bom yes) (on_board yes) (fields_autoplaced)
-    (property "Reference" "Q?" (id 0) (at 116.84 79.3749 0)
+    (property "Reference" "Q2" (id 0) (at 116.84 79.3749 0)
       (effects (font (size 1.27 1.27)) (justify left))
     )
@@
   (symbol (lib_id "JRIX Transistor:SIA931DJ") (at 81.915 88.9 270) (unit 2)
     (in_bom yes) (on_board yes) (fields_autoplaced)
-    (property "Reference" "Q?" (id 0) (at 81.915 100.965 90))
+    (property "Reference" "Q1" (id 0) (at 81.915 100.965 90))
     (property "Value" "SIA931DJ" (id 1) (at 81.915 103.505 90))
-    (property "Footprint" "" (id 2) (at 89.535 73.66 0)
+    (property "Footprint" "Package_TO_SOT_SMD:SOT-363_SC-70-6" (id 2) (at 89.535 73.66 0)
       (effects (font (size 1.27 1.27)) hide)
     )
@@
   (symbol (lib_id "JRIX Comparators:NCS2202A") (at 54.61 38.735 270) (unit 2)
     (in_bom yes) (on_board yes) (fields_autoplaced)
-    (property "Reference" "U?" (id 0) (at 56.515 42.5449 90)
+    (property "Reference" "U11" (id 0) (at 56.515 42.5449 90)
       (effects (font (size 1.27 1.27)) (justify left))
     )
@@
       (effects (font (size 1.27 1.27)) (justify left))
     )
-    (property "Footprint" "" (id 2) (at 62.23 17.145 0)
+    (property "Footprint" "JRIX UDFN Footprints:Package_UDFN-6_1.2x1.0mm_P0.4" (id 2) (at 62.23 17.145 0)
       (effects (font (size 1.27 1.27)) hide)
     )
@@
     (pin "6")
     (pin "1")
+    (pin "2")
     (pin "5")
   )
   (symbol (lib_id "JRIX Comparators:NCS2202A") (at 48.895 75.565 0) (unit 1)
     (in_bom yes) (on_board yes) (fields_autoplaced)
-    (property "Reference" "U?" (id 0) (at 59.055 70.485 0))
+    (property "Reference" "U11" (id 0) (at 59.055 70.485 0))
     (property "Value" "NCS2202A" (id 1) (at 59.055 73.025 0))
-    (property "Footprint" "" (id 2) (at 27.305 67.945 0)
+    (property "Footprint" "JRIX UDFN Footprints:Package_UDFN-6_1.2x1.0mm_P0.4" (id 2) (at 27.305 67.945 0)
       (effects (font (size 1.27 1.27)) hide)
     )
@@
     (pin "6")
     (pin "1")
-    (pin "5")
-  )
+    (pin "2")
+    (pin "5")
+  )
